File: PCB/v1.1/tarocco.sch (EAGLE design)
At the start: 42 parts, among them IC1 CY8C4545PVI, Q1 NEXFET_SINGLECSD18537NQ5A, Q2 NEXFET_SINGLECSD18537NQ5A, Q3 NEXFET_SINGLECSD18537NQ5A, Q4 NEXFET_SINGLECSD18537NQ5A

Commit message: august updates
Parts:
- removed PGRM: (no value), SparkFun-Connectors:M05SMD2
- added TP1, TP2, TP3, TP4, TP5: TEST-POINT3X5, SparkFun-Passives:TEST-POINT3X5
- added U$1, U$3: FIDUCIAL, adafruit:FIDUCIAL
Connections:
- removed net N$46: IC1.P0.2
- removed net N$47: IC1.P0.3
- removed net N$48: IC1.P0.6
- removed net N$49: IC1.P0.7
- net 5V: now also TP4.1; no longer PGRM.4
- net DIRECTION: now also IC1.P0.7; no longer IC1.P4.3
- net ERROR: now also IC1.P0.2; no longer IC1.P4.0
- net GND: now also TP5.1; no longer PGRM.5
- net RESET: now also IC1.P0.3; no longer IC1.P4.1
- net STEP: now also IC1.P0.6; no longer IC1.P4.2
- net SWDCLK: now also TP2.1; no longer PGRM.2
- net SWDIO: now also TP3.1; no longer PGRM.3
- net XRES: now also TP1.1; no longer PGRM.1
Changed lines of the file:
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@@
 <layer number="94" name="Symbols" color="4" fill="1" visible="yes" active="yes"/>
 <layer number="95" name="Names" color="7" fill="1" visible="yes" active="yes"/>
-<layer number="96" name="Values" color="7" fill="1" visible="no" active="yes"/>
+<layer number="96" name="Values" color="7" fill="1" visible="yes" active="yes"/>
 <layer number="97" name="Info" color="7" fill="1" visible="no" active="yes"/>
 <layer number="98" name="Guide" color="6" fill="1" visible="no" active="yes"/>
@@
 <part name="GND6" library="SparkFun-Aesthetics" deviceset="GND" device=""/>
 <part name="GND8" library="SparkFun-Aesthetics" deviceset="GND" device=""/>
-<part name="PGRM" library="SparkFun-Connectors" deviceset="M05" device="SMD2"/>
 <part name="GND9" library="SparkFun-Aesthetics" deviceset="GND" device=""/>
 <part name="C11" library="adafruit" deviceset="C-US" device="C0603" value="100n"/>
+<part name="TP1" library="SparkFun-Passives" deviceset="TEST-POINT" device="3X5"/>
+<part name="TP2" library="SparkFun-Passives" deviceset="TEST-POINT" device="3X5"/>
+<part name="TP3" library="SparkFun-Passives" deviceset="TEST-POINT" device="3X5"/>
+<part name="TP4" library="SparkFun-Passives" deviceset="TEST-POINT" device="3X5"/>
+<part name="TP5" library="SparkFun-Passives" deviceset="TEST-POINT" device="3X5"/>
+<part name="U$1" library="adafruit" deviceset="FIDUCIAL" device=""/>
+<part name="U$3" library="adafruit" deviceset="FIDUCIAL" device=""/>
 </parts>
 <sheets>
@@
 <instance part="GND6" gate="1" x="17.78" y="58.42"/>
 <instance part="GND8" gate="1" x="116.84" y="111.76"/>
-<instance part="PGRM" gate="G$1" x="15.24" y="40.64" rot="MR180"/>
 <instance part="GND9" gate="1" x="25.4" y="30.48"/>
 <instance part="C11" gate="G$1" x="25.4" y="76.2" smashed="yes">
@@
 <attribute name="VALUE" x="26.416" y="72.009" size="1.778" layer="96"/>
 </instance>
+<instance part="TP1" gate="G$1" x="22.86" y="45.72" smashed="yes" rot="R180"/>
+<instance part="TP2" gate="G$1" x="22.86" y="43.18" smashed="yes" rot="R180"/>
+<instance part="TP3" gate="G$1" x="22.86" y="40.64" smashed="yes" rot="R180"/>
+<instance part="TP4" gate="G$1" x="22.86" y="38.1" smashed="yes" rot="R180"/>
+<instance part="TP5" gate="G$1" x="22.86" y="35.56" smashed="yes" rot="R180"/>
+<instance part="U$1" gate="G$1" x="0" y="127"/>
+<instance part="U$3" gate="G$1" x="0" y="119.38"/>
 </instances>
 <busses>
@@
 </segment>
 <segment>
-<pinref part="PGRM" gate="G$1" pin="5"/>
 <pinref part="GND9" gate="1" pin="GND"/>
 <wire x1="22.86" y1="35.56" x2="25.4" y2="35.56" width="0.1524" layer="91"/>
 <wire x1="25.4" y1="35.56" x2="25.4" y2="33.02" width="0.1524" layer="91"/>
+<pinref part="TP5" gate="G$1" pin="1"/>
 </segment>
 </net>
@@
 </segment>
 <segment>
-<pinref part="PGRM" gate="G$1" pin="4"/>
 <wire x1="22.86" y1="38.1" x2="25.4" y2="38.1" width="0.1524" layer="91"/>
 <label x="22.86" y="38.1" size="1.778" layer="95"/>
+<pinref part="TP4" gate="G$1" pin="1"/>
 </segment>
 </net>
@@
 </segment>
 <segment>
-<pinref part="IC1" gate="G$1" pin="P4.0"/>
-<wire x1="86.36" y1="55.88" x2="91.44" y2="55.88" width="0.1524" layer="91"/>
-<label x="88.9" y="55.88" size="1.778" layer="95"/>
+<pinref part="IC1" gate="G$1" pin="P0.2"/>
+<wire x1="86.36" y1="71.12" x2="91.44" y2="71.12" width="0.1524" layer="91"/>
+<label x="88.9" y="71.12" size="1.778" layer="95"/>
 </segment>
 </net>
@@
 </segment>
 <segment>
-<pinref part="IC1" gate="G$1" pin="P4.1"/>
-<wire x1="86.36" y1="58.42" x2="91.44" y2="58.42" width="0.1524" layer="91"/>
-<label x="88.9" y="58.42" size="1.778" layer="95"/>
+<pinref part="IC1" gate="G$1" pin="P0.3"/>
+<wire x1="86.36" y1="73.66" x2="91.44" y2="73.66" width="0.1524" layer="91"/>
+<label x="88.9" y="73.66" size="1.778" layer="95"/>
 </segment>
 </net>
@@
 </segment>
 <segment>
-<pinref part="IC1" gate="G$1" pin="P4.2"/>
-<wire x1="86.36" y1="60.96" x2="91.44" y2="60.96" width="0.1524" layer="91"/>
-<label x="88.9" y="60.96" size="1.778" layer="95"/>
+<pinref part="IC1" gate="G$1" pin="P0.6"/>
+<wire x1="86.36" y1="76.2" x2="91.44" y2="76.2" width="0.1524" layer="91"/>
+<label x="88.9" y="76.2" size="1.778" layer="95"/>
 </segment>
 </net>
@@
 </segment>
 <segment>
-<pinref part="IC1" gate="G$1" pin="P4.3"/>
-<wire x1="86.36" y1="63.5" x2="91.44" y2="63.5" width="0.1524" layer="91"/>
-<label x="88.9" y="63.5" size="1.778" layer="95"/>
+<pinref part="IC1" gate="G$1" pin="P0.7"/>
+<wire x1="86.36" y1="78.74" x2="91.44" y2="78.74" width="0.1524" layer="91"/>
+<label x="88.9" y="78.74" size="1.778" layer="95"/>
 </segment>
 </net>
@@
 </segment>
 <segment>
-<pinref part="PGRM" gate="G$1" pin="3"/>
 <wire x1="22.86" y1="40.64" x2="25.4" y2="40.64" width="0.1524" layer="91"/>
 <label x="22.86" y="40.64" size="1.778" layer="95"/>
+<pinref part="TP3" gate="G$1" pin="1"/>
 </segment>
 </net>
@@
 </segment>
 <segment>
-<pinref part="PGRM" gate="G$1" pin="2"/>
 <wire x1="22.86" y1="43.18" x2="25.4" y2="43.18" width="0.1524" layer="91"/>
 <label x="22.86" y="43.18" size="1.778" layer="95"/>
-</segment>
-</net>
-<net name="N$46" class="0">
-<segment>
-<pinref part="IC1" gate="G$1" pin="P0.2"/>
-<wire x1="86.36" y1="71.12" x2="91.44" y2="71.12" width="0.1524" layer="91"/>
-</segment>
-</net>
-<net name="N$47" class="0">
-<segment>
-<pinref part="IC1" gate="G$1" pin="P0.3"/>
-<wire x1="86.36" y1="73.66" x2="91.44" y2="73.66" width="0.1524" layer="91"/>
-</segment>
-</net>
-<net name="N$48" class="0">
-<segment>
-<pinref part="IC1" gate="G$1" pin="P0.6"/>
-<wire x1="86.36" y1="76.2" x2="91.44" y2="76.2" width="0.1524" layer="91"/>
-</segment>
-</net>
-<net name="N$49" class="0">
-<segment>
-<pinref part="IC1" gate="G$1" pin="P0.7"/>
-<wire x1="86.36" y1="78.74" x2="91.44" y2="78.74" width="0.1524" layer="91"/>
+<pinref part="TP2" gate="G$1" pin="1"/>
 </segment>
 </net>
@@
 </segment>
 <segment>
-<pinref part="PGRM" gate="G$1" pin="1"/>
 <wire x1="22.86" y1="45.72" x2="25.4" y2="45.72" width="0.1524" layer="91"/>
 <label x="22.86" y="45.72" size="1.778" layer="95"/>
-</segment>
-</net>
+<pinref part="TP1" gate="G$1" pin="1"/>
+</segment>
+</net>
