File: PCB/v1.1/tarocco-v1.1.sch (EAGLE design)
At the start: 48 parts, among them IC1 CY8C4545PVI, Q1 NEXFET_SINGLECSD18537NQ5A, Q2 NEXFET_SINGLECSD18537NQ5A, Q3 NEXFET_SINGLECSD18537NQ5A, Q4 NEXFET_SINGLECSD18537NQ5A

Commit message: updated pcb files
Other:
- note added: "CY8C4245PVI"
Changed lines of the file:
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@@
 <sheet>
 <plain>
+<text x="48.26" y="50.8" size="1.778" layer="95">CY8C4245PVI</text>
 </plain>
 <instances>
@@
 <attribute name="VALUE" x="155.448" y="69.85" size="1.778" layer="96" rot="R270"/>
 </instance>
-<instance part="IC1" gate="G$1" x="66.04" y="73.66" smashed="yes">
-<attribute name="VALUE" x="50.8" y="50.8" size="1.778" layer="96"/>
-</instance>
+<instance part="IC1" gate="G$1" x="66.04" y="73.66" smashed="yes"/>
 <instance part="SERIAL" gate="A" x="106.68" y="121.92"/>
 <instance part="GND6" gate="1" x="17.78" y="58.42"/>
